File: hardware/e1-xcvr/e1_xcvr.brd (EAGLE design)
At the start: 70 x 60 mm, 48 parts, among them T1 BC847C, U1 IDT82V2081, U3_2M 2.048 Mhz, U4_1M5 1.544 MHz, U6 TPS736XX

Commit message: e1_xcvr: Give signals proper names
Change-Id: I04107430cab02e493bbabef60b1cc19b535caad6
Connections:
- net N$15 renamed TDP
- net N$16 renamed TDN
- net N$17 renamed !RST
- net N$19 renamed SDI
- net N$2 renamed RDN
- net N$20 renamed !CS
- net N$21 renamed SDO
- net N$22 renamed SCLK
- net N$24 renamed !INT
- net N$3 renamed RDP
- net N$4 renamed RCLK
- net N$7 renamed _VIN
Changed lines of the file:
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@@
 <wire x1="28.9475" y1="36.3525" x2="30.0025" y2="36.3525" width="0.4064" layer="1"/>
 </signal>
-<signal name="N$2">
+<signal name="RDN">
 <contactref element="U1" pad="6"/>
 <contactref element="JP2" pad="10"/>
@@
 <via x="37.94" y="19.8425" extent="1-16" drill="0.6"/>
 </signal>
-<signal name="N$3">
+<signal name="RDP">
 <contactref element="U1" pad="5"/>
 <contactref element="JP2" pad="8"/>
@@
 <via x="36.9875" y="18.255" extent="1-16" drill="0.6"/>
 </signal>
-<signal name="N$4">
+<signal name="RCLK">
 <contactref element="U1" pad="4"/>
 <contactref element="JP2" pad="6"/>
@@
 <wire x1="42.0675" y1="17.62" x2="43.9725" y2="17.62" width="0.3048" layer="16"/>
 </signal>
-<signal name="N$15">
+<signal name="TDP">
 <contactref element="U1" pad="2"/>
 <contactref element="JP2" pad="7"/>
@@
 <via x="34.13" y="18.89" extent="1-16" drill="0.6"/>
 </signal>
-<signal name="N$16">
+<signal name="TDN">
 <contactref element="U1" pad="3"/>
 <contactref element="JP2" pad="5"/>
@@
 <via x="35.4" y="19.8425" extent="1-16" drill="0.6"/>
 </signal>
-<signal name="N$17">
+<signal name="!RST">
 <contactref element="U1" pad="12"/>
 <contactref element="JP2" pad="2"/>
@@
 <wire x1="16.8625" y1="39.7225" x2="18.255" y2="41.115" width="0.4064" layer="1"/>
 </signal>
-<signal name="N$22">
+<signal name="SCLK">
 <contactref element="JP1" pad="9"/>
 <contactref element="U1" pad="25"/>
@@
 <wire x1="52.6475" y1="53.4975" x2="51.5925" y2="53.4975" width="0.3048" layer="1"/>
 </signal>
-<signal name="N$19">
+<signal name="SDI">
 <contactref element="U1" pad="24"/>
 <contactref element="JP1" pad="8"/>
@@
 <via x="39.845" y="28.7325" extent="1-16" drill="0.6"/>
 </signal>
-<signal name="N$20">
+<signal name="!CS">
 <contactref element="JP1" pad="10"/>
 <contactref element="U1" pad="21"/>
@@
 <via x="44.925" y="30.32" extent="1-16" drill="0.6"/>
 </signal>
-<signal name="N$21">
+<signal name="SDO">
 <contactref element="U1" pad="23"/>
 <contactref element="JP1" pad="7"/>
@@
 <wire x1="41.305" y1="28.605" x2="40.7975" y2="28.0975" width="0.3048" layer="1"/>
 </signal>
-<signal name="N$24">
+<signal name="!INT">
 <contactref element="U1" pad="20"/>
 <contactref element="JP1" pad="4"/>
@@
 <via x="38.8925" y="27.145" extent="1-16" drill="0.6"/>
 </signal>
-<signal name="N$7" class="1">
+<signal name="_VIN" class="1">
 <contactref element="JP1" pad="1"/>
 <contactref element="SJ2" pad="2"/>
