File: hardware/e1-xcvr/e1_xcvr.sch (EAGLE design)
At the start: 48 parts, among them T1 BC847C, U1 IDT82V2081, U3_2M 2.048 Mhz, U4_1M5 1.544 MHz, U6 TPS736XX

Commit message: e1_xcvr: Give signals proper names
Change-Id: I04107430cab02e493bbabef60b1cc19b535caad6
Connections:
- net N$15 renamed TDP
- net N$16 renamed TDN
- net N$17 renamed !RST
- net N$19 renamed SDI
- net N$2 renamed RDN
- net N$20 renamed !CS
- net N$21 renamed SDO
- net N$22 renamed SCLK
- net N$24 renamed !INT
- net N$3 renamed RDP
- net N$4 renamed RCLK
- net N$7 renamed _VIN
Changed lines of the file:
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@@
 <grid distance="0.1" unitdist="inch" unit="inch" style="lines" multiple="1" display="no" altdistance="0.01" altunitdist="inch" altunit="inch"/>
 <layers>
-<layer number="1" name="Top" color="4" fill="1" visible="yes" active="no"/>
-<layer number="2" name="Route2" color="1" fill="3" visible="yes" active="no"/>
-<layer number="3" name="Route3" color="4" fill="3" visible="yes" active="no"/>
-<layer number="14" name="Route14" color="1" fill="6" visible="yes" active="no"/>
-<layer number="15" name="Route15" color="4" fill="6" visible="yes" active="no"/>
-<layer number="16" name="Bottom" color="1" fill="1" visible="yes" active="no"/>
-<layer number="17" name="Pads" color="2" fill="1" visible="yes" active="no"/>
-<layer number="18" name="Vias" color="2" fill="1" visible="yes" active="no"/>
-<layer number="19" name="Unrouted" color="6" fill="1" visible="yes" active="no"/>
-<layer number="20" name="Dimension" color="15" fill="1" visible="yes" active="no"/>
-<layer number="21" name="tPlace" color="7" fill="1" visible="yes" active="no"/>
-<layer number="22" name="bPlace" color="7" fill="1" visible="yes" active="no"/>
-<layer number="23" name="tOrigins" color="15" fill="1" visible="yes" active="no"/>
-<layer number="24" name="bOrigins" color="15" fill="1" visible="yes" active="no"/>
-<layer number="25" name="tNames" color="7" fill="1" visible="yes" active="no"/>
-<layer number="26" name="bNames" color="7" fill="1" visible="yes" active="no"/>
-<layer number="27" name="tValues" color="7" fill="1" visible="yes" active="no"/>
-<layer number="28" name="bValues" color="7" fill="1" visible="yes" active="no"/>
+<layer number="1" name="Top" color="4" fill="1" visible="no" active="no"/>
+<layer number="2" name="Route2" color="1" fill="3" visible="no" active="no"/>
+<layer number="3" name="Route3" color="4" fill="3" visible="no" active="no"/>
+<layer number="14" name="Route14" color="1" fill="6" visible="no" active="no"/>
+<layer number="15" name="Route15" color="4" fill="6" visible="no" active="no"/>
+<layer number="16" name="Bottom" color="1" fill="1" visible="no" active="no"/>
+<layer number="17" name="Pads" color="2" fill="1" visible="no" active="no"/>
+<layer number="18" name="Vias" color="2" fill="1" visible="no" active="no"/>
+<layer number="19" name="Unrouted" color="6" fill="1" visible="no" active="no"/>
+<layer number="20" name="Dimension" color="15" fill="1" visible="no" active="no"/>
+<layer number="21" name="tPlace" color="7" fill="1" visible="no" active="no"/>
+<layer number="22" name="bPlace" color="7" fill="1" visible="no" active="no"/>
+<layer number="23" name="tOrigins" color="15" fill="1" visible="no" active="no"/>
+<layer number="24" name="bOrigins" color="15" fill="1" visible="no" active="no"/>
+<layer number="25" name="tNames" color="7" fill="1" visible="no" active="no"/>
+<layer number="26" name="bNames" color="7" fill="1" visible="no" active="no"/>
+<layer number="27" name="tValues" color="7" fill="1" visible="no" active="no"/>
+<layer number="28" name="bValues" color="7" fill="1" visible="no" active="no"/>
 <layer number="29" name="tStop" color="7" fill="3" visible="no" active="no"/>
 <layer number="30" name="bStop" color="7" fill="6" visible="no" active="no"/>
@@
 <layer number="35" name="tGlue" color="7" fill="4" visible="no" active="no"/>
 <layer number="36" name="bGlue" color="7" fill="5" visible="no" active="no"/>
-<layer number="37" name="tTest" color="7" fill="1" visible="yes" active="no"/>
-<layer number="38" name="bTest" color="7" fill="1" visible="yes" active="no"/>
+<layer number="37" name="tTest" color="7" fill="1" visible="no" active="no"/>
+<layer number="38" name="bTest" color="7" fill="1" visible="no" active="no"/>
 <layer number="39" name="tKeepout" color="4" fill="11" visible="no" active="no"/>
 <layer number="40" name="bKeepout" color="1" fill="11" visible="no" active="no"/>
@@
 <layer number="44" name="Drills" color="7" fill="1" visible="no" active="no"/>
 <layer number="45" name="Holes" color="7" fill="1" visible="no" active="no"/>
-<layer number="46" name="Milling" color="3" fill="1" visible="yes" active="no"/>
-<layer number="47" name="Measures" color="7" fill="1" visible="yes" active="no"/>
-<layer number="48" name="Document" color="7" fill="1" visible="yes" active="no"/>
-<layer number="49" name="Reference" color="7" fill="1" visible="yes" active="no"/>
-<layer number="51" name="tDocu" color="7" fill="1" visible="yes" active="no"/>
-<layer number="52" name="bDocu" color="7" fill="1" visible="yes" active="no"/>
+<layer number="46" name="Milling" color="3" fill="1" visible="no" active="no"/>
+<layer number="47" name="Measures" color="7" fill="1" visible="no" active="no"/>
+<layer number="48" name="Document" color="7" fill="1" visible="no" active="no"/>
+<layer number="49" name="Reference" color="7" fill="1" visible="no" active="no"/>
+<layer number="51" name="tDocu" color="7" fill="1" visible="no" active="no"/>
+<layer number="52" name="bDocu" color="7" fill="1" visible="no" active="no"/>
 <layer number="91" name="Nets" color="2" fill="1" visible="yes" active="yes"/>
 <layer number="92" name="Busses" color="1" fill="1" visible="yes" active="yes"/>
@@
 </segment>
 </net>
-<net name="N$2" class="0">
+<net name="RDN" class="0">
 <segment>
 <pinref part="U1" gate="G$1" pin="CV/RDN"/>
@@
 </segment>
 </net>
-<net name="N$3" class="0">
+<net name="RDP" class="0">
 <segment>
 <pinref part="U1" gate="G$1" pin="RD/RDP"/>
@@
 </segment>
 </net>
-<net name="N$4" class="0">
+<net name="RCLK" class="0">
 <segment>
 <pinref part="U1" gate="G$1" pin="RCLK"/>
@@
 </segment>
 </net>
-<net name="N$15" class="0">
+<net name="TDP" class="0">
 <segment>
 <pinref part="U1" gate="G$1" pin="TD/TDP"/>
@@
 </segment>
 </net>
-<net name="N$16" class="0">
+<net name="TDN" class="0">
 <segment>
 <pinref part="U1" gate="G$1" pin="TDN"/>
@@
 </segment>
 </net>
-<net name="N$17" class="0">
+<net name="!RST" class="0">
 <segment>
 <pinref part="U1" gate="G$4" pin="!RST"/>
@@
 </segment>
 </net>
-<net name="N$22" class="0">
+<net name="SCLK" class="0">
 <segment>
 <wire x1="5.08" y1="71.12" x2="5.08" y2="76.2" width="0.1524" layer="91"/>
@@
 </segment>
 </net>
-<net name="N$19" class="0">
+<net name="SDI" class="0">
 <segment>
 <pinref part="U1" gate="G$3" pin="SDI/WR/RW"/>
@@
 </segment>
 </net>
-<net name="N$20" class="0">
+<net name="!CS" class="0">
 <segment>
 <pinref part="JP1" gate="A" pin="10"/>
@@
 </segment>
 </net>
-<net name="N$21" class="0">
+<net name="SDO" class="0">
 <segment>
 <pinref part="U1" gate="G$3" pin="SDO/!ACK/RDY"/>
@@
 </segment>
 </net>
-<net name="N$24" class="0">
+<net name="!INT" class="0">
 <segment>
 <pinref part="U1" gate="G$3" pin="!INT"/>
@@
 </segment>
 </net>
-<net name="N$7" class="1">
+<net name="_VIN" class="1">
 <segment>
 <pinref part="JP1" gate="A" pin="1"/>
