File: hardware/e1-tracer/e1-tracer.sch (EAGLE design)
At the start: 118 parts, among them IC1 MCP1703T-1202E/CB, IC2 W25Q80DVSNIG, IC3 TLV70233DBVR, IC4 ASEM1-12.000MHZ-LC-T, J1 PASSTHROUGH, M1 MENTOR_12701001, M2 MENTOR_12701001, SW1 TACTSW-TL3340, T1 BC847C, T2 BC847C, U1 ICE40UP5K-SG48I, U2 IP4234CZ6, U3 IP4234CZ6, U4 IDT82V2081, U5 IDT82V2081, U6 2.048 Mhz, U7 1.544 MHz, X1 MINI-USB-SHIELD-UX60-MB-5ST, X2 JACK2.5_SJ-2523

Commit message: e1-tracer: solve everything towards v2
* retract light guides and RJ45 1.5mm inwards (solves SYS#5051)
* SPI MOSI/MISO mismatch fixed (solves SYS#5050)
* footpint mismatch to BOM for L3,L4 fixed (solves SYS#5053)
* PCB had to get 5mm slimmer (adresses SYS#5088)
* repaired silk on name bott side
* DRC

Change-Id: I97ab7240b9b1fb68347dc994885c926b8c192217
Parts:
- L2, L3: device inductor-neosid:SM-1206 -> rc-sysmocom:INDUCTOR0805
Connections:
- net IOB_32A_SPI_SO: now also IC2.SI(D0); no longer IC2.SO(D1)
- net IOB_33B_SPI_SI: now also IC2.SO(D1); no longer IC2.SI(D0)

Commit message: e1-tracer: update BOM attributes to 1st v2 prod run parts
* L2, L3 now 0805
* R6, R7 now 0402
* IC4 now ASEMB-12.000MHZ-LC-T
* RoHS state enabled again in scraper, not yet used in BOM

Change-Id: I4f1a82476ca84552efd71a47231e8b6ac02a3358
Parts:
- C25, C26, C27, C28, CDONE, D1, D2, D3, D4, D5, D6, D7, D8, IC1, IC2, IC3, L2, L3, LOS1, LOS2, PWR, R1, R10, R13, R14, R15, R16, R17, R18, R19, R2, R20, R21, R22, R23, R24, R25, R26, R27, R28, R29, R3, R30, R31, R32, R33, R34, R35, R36, R37, R38, R39, R4, R40, R41, R42, R43, R44, R45, R46, R5, R8, R9, T1, T2, U1: ROHSCERTIFICATE UNKNOWN ROHS CERTIFICATE -> RoHS3-konform
- IC4: value ASEM1-12.000MHZ-LC-T -> ASEMB-12.000MHZ-LC-T; CLASS IC / XTAL / XO -> UNKNOWN CLASS; LINK https://www.digikey.de/product-detail/de/abracon-llc/ASEM1-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 -> https://www.digikey.de/product-detail/de/abracon-llc/ASEMB-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; MANUFACTURERPARTNUMBER ASEM1-12.000MHZ-LC-T -> ASEMB-12.000MHZ-LC-T; ROHSCERTIFICATE UNKNOWN ROHS CERTIFICATE -> RoHS-konform; SOURCEPARTNUMBER 535-9757-1-ND -> 535-11744-1-ND
- J1, LED1, TR1, TR2: ROHSCERTIFICATE UNKNOWN ROHS CERTIFICATE -> RoHS-konform
- R6, R7: DESCRIPTION RES 33 OHM 5%% 1/10W 0603 -> RES SMD 33 OHM 1%% 1/16W 0402; LINK https://www.digikey.de/product-detail/de/stackpole-electron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 -> https://www.digikey.de/product-detail/de/yageo/RC0402FR-073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; MANUFACTURER Stackpole Electronics Inc -> Yageo; MANUFACTURERPARTNUMBER RMCF0603JT33R0 -> RC0402FR-0733RL; ROHSCERTIFICATE UNKNOWN ROHS CERTIFICATE -> RoHS3-konform; SOURCEPARTNUMBER RMCF0603JT33R0CT-ND -> 311-33.0LRCT-ND
- U4, U5, U6: MANUFACTURER Renesas Electronics America Inc. -> Renesas Electronics America Inc; ROHSCERTIFICATE UNKNOWN ROHS CERTIFICATE -> RoHS3-konform
